Commit message: [REF] Port the driver to ROS2 Jazzy - tested on FT150

File: robotiq_ft_sensor_description/urdf/robotiq_ft300.urdf.xacro (robot description, xacro)
@@ -55,5 +55,5 @@
             <child link="${tf_prefix}ft300_sensor" />
         </joint>
-        <joint name="${tf_prefix}measurment_joint" type="fixed">
+        <joint name="${tf_prefix}measurement_joint" type="fixed">
             <origin xyz="0 0 0" rpy="0 ${pi} ${-pi/2}" />
             <parent link="${tf_prefix}ft300_sensor" />

File: robotiq_ft_sensor_description/urdf/robotiq_fts150.urdf.xacro (robot description, xacro)
@@ -30,5 +30,5 @@
         </link>
         <!-- virtual measurement frame -->
-        <joint name="${tf_prefix}measurment_joint" type="fixed" >
+        <joint name="${tf_prefix}measurement_joint" type="fixed" >
             <origin xyz="0 0 0.01625" rpy="0 0 0" />
             <parent link="${tf_prefix}fts_robotside" />
